File: Cibike_PWM.X/docs/1379_control.sch (EAGLE design)
At the start: 179 parts, among them Q1 ZXMN6A08E6, Q10 ZXMP3A17E6, Q11 ZXMP3A17E6, Q12 ZXMP3A17E6, Q2 ZXMN6A08E6, Q3 IRLML0100TR, Q4 ZXMP3A17E6, Q5 ZXMP3A17E6, Q6 ZXMP3A17E6, Q7 ZXMP3A17E6, Q8 ZXMP3A17E6, Q9 ZXMP3A17E6, T1 2N7002A, T2 2N7002A, T3 2N7002A, T4 2N7002A, U1 AP3031, U10 ST-M24256E-FMN6TP, U11 AP3031, U12 AP3031, U13 AP3031, U14 AP3031, U2 ZXLD1370Q, U3 AP3031, U4 AP3031, U5 AP3031, U6 ZXLD1370Q, U7 PCA9685PW,118, U8 PIC32MX120F064H, U9 LMR51420, X1 ENODER_ROTARY, X2 BM05B-PASS, X3 ENCODER-2, Y1 MCSJK-3N-8.00-3.3-25-B

Commit message: New layout
Parts:
- removed D2, D4: (no value), zetex:DSOT23
- removed R23: 2k7, rcl:R-EU_R0603
- removed R35, R36: 4k7, rcl:R-EU_R0603
- removed R51: 10k, rcl:R-EU_R0603
- removed T1, T2, T4: 2N7002A, zetex:NMOSSOT23
- added C58: 10p, rcl:C-EUC0603
- added JP1: (no value), pinhead:PINHD-1X4
- added JP2, JP5: (no value), pinhead:PINHD-1X8
- added JP3: (no value), pinhead:PINHD-1X11
- added R45: 1k, rcl:R-EU_R0603
- added S4, S6: (no value), SparkFun-Switches:SWITCH-SPDT-PTH-11.6X4.0MM
- added S7: DPDT, untitled:DPDT
- C25: device rcl:C-EUC0805 -> rcl:C-EUC0603
- R1, R10, R11, R19: device rcl:R-EU_R0603 -> rcl:R-EU_R0805
- R14: device rcl:R-EU_R0805 -> rcl:R-EU_R0603
- R22: value 0R -> 2R2
- R8: value 2k7 -> 10k
- S2: value MOMENTARY-SWITCH-SPST-SMD-6.2MM-TALL -> MOMENTARY-SWITCH-SPST-PTH-6.0MM; device SparkFun-Switches:MOMENTARY-SWITCH-SPST-SMD-6.2MM-TALL -> SparkFun-Switches:MOMENTARY-SWITCH-SPST-PTH-6.0MM
Connections:
- removed net N$13: U11.CTRL, U12.CTRL, U13.CTRL, U14.CTRL, U4.CTRL
- removed net OVP/PWM_TI: T2.D, T4.D, U6.PWM
- removed net PWM1: RN1A.1
- removed net PWM2: RN1B.1
- removed net PWM3: RN1C.1
- removed net PWM4: RN1D.1
- removed net PWM5: RN2A.1
- removed net PWM6: RN2B.1
- removed net PWM7: RN2C.1
- removed net TI_PWM: Q3.G
- removed net VIN: Q8.D
- removed net V_TAIL_LOW_A: C24.1, D6.C
- removed net V_TAIL_LOW_K: R11.1, U5.FB
- removed net V_TAIL_UPP_A: C22.1, D5.C
- removed net V_TAIL_UPP_K: R10.1, U4.FB
- new net CTRL1: S7.2, U3.CTRL
- new net CTRL2: S7.5, U1.CTRL
- new net N$65: C58.2, R45.1
- new net N$67: Q3.G, S6.P
- new net PWM_CHMSL: RN2C.1, U14.CTRL
- new net PWM_LET: RN2B.1, U13.CTRL
- new net PWM_TAIL_LOW: RN2A.1, U5.CTRL
- new net PWM_TAIL_UPP: RN1C.1, U4.CTRL
- new net TAIL_LOW_A: C24.1, D6.C, JP3.10
- new net TAIL_LOW_K: JP3.9, R11.1, U5.FB
- new net TAIL_UPP_A: C22.1, D5.C, JP3.8
- new net TAIL_UPP_K: JP3.7, R10.1, U4.FB
- new net VCC: JP2.8, Q8.D
- new net V_TAIL1: C13.2, C14.2, C7.2, R5.1, R9.1, S4.P, U2.VAUX, U2.VIN
- net 3,3V: now also JP1.1; no longer R35.1, R36.1
- net CHMSL: now also JP2.7
- net CHMSL_A: now also JP5.8; no longer U14.OV
- net CHMSL_K: now also JP5.7
- net FOG: now also JP2.4
- net FOG_A: now also JP5.2; no longer U11.OV
- net FOG_K: now also JP5.1
- net FREQ/DUTY: now also U8.RB7; no longer U8.RB9
- net GND: now also C58.1, JP1.2, JP3.4; no longer R23.1, R51.1, R8.1, T1.S, T2.S, T4.S
- net LET: now also JP2.6
- net LET_A: now also JP5.4; no longer U13.OV
- net LET_K: now also JP5.3
- net LOCK: now also U8.RB6; no longer U8.RB5
- net N$10: now also R8.1, S6.S; no longer D4.A, R8.2, T1.G
- net N$14: now also U11.CTRL; no longer U5.CTRL
- net N$25: now also R45.2
- net N$33: now also U12.CTRL; no longer D2.A, R23.2, T2.G
- net OVP/PWM_TAIL_MID: no longer T1.D
- net P1: now also U8.RF4; no longer U8.RB12
- net PWM_T/B_LOW: now also RN1B.1, S7.6; no longer U1.CTRL
- net PWM_T/B_UPP: now also RN1A.1, S7.3; no longer U3.CTRL
- net PWM_TAIL_MID: now also RN1D.1
- net PWM_TI: now also S6.O; no longer R51.2, T4.G
- net RESET: now also U8.RB9; no longer U8.RB11
- net REV: now also JP2.5
- net REV_A: now also JP5.6; no longer U12.OV
- net REV_K: now also JP5.5
- net ROT_+: now also U8.RB12; no longer U8.RB6
- net ROT_-: now also U8.RB11; no longer U8.RB7
- net SCL: now also JP1.3; no longer R35.2
- net SDA: now also JP1.4; no longer R36.2
- net T/B: now also JP2.2
- net T/B_LOW_OUT_A: now also JP3.6
- net T/B_LOW_OUT_K: now also JP3.5
- net T/B_UPP_OUT_A: now also JP3.3
- net T/B_UPP_OUT_K: now also JP3.1
- net TAIL: now also JP2.3
- net TAIL_MID_A: now also JP3.11; no longer D4.C
- net TI: now also JP2.1
- net TI_A: now also JP3.2; no longer D2.C
- net V_T/B: now also S7.1, S7.4
- net V_TAIL: now also S4.S; no longer C13.2, C14.2, C7.2, R5.1, R9.1, U2.VAUX, U2.VIN
- net V_TI: now also R8.2
Other:
- note added: "16CH I2C Extender"
- note added: "3,3V Source"
- note added: "CLOCK"
- note added: "D4 = 49V for Outer"
- note added: "I2C EEPROM"
- note added: "MCU"
